Commit message: updated changes

File: mybot_description/urdf/macros.xacro (robot description, xacro)
@@ -1,2 +1,3 @@
+<?xml version="1.0"?>
 <robot>
 <macro name="cylinder_inertia" params="m r h">
@@ -19,48 +20,50 @@
 </macro>
 <macro name="wheel" params="lr tY">
-<link name="${lr}_wheel">
-  <collision>
-    <origin xyz="0 0 0" rpy="0 ${PI/2} ${PI/2}" />
-    <geometry>
-      <cylinder length="${wheelWidth}" radius="${wheelRadius}"/>
-    </geometry>
-  </collision>
-  <visual>
-    <origin xyz="0 0 0" rpy="0 ${PI/2} ${PI/2}" />
-    <geometry>
-      <cylinder length="${wheelWidth}" radius="${wheelRadius}"/>
-    </geometry>
-    <material name="black"/>
-  </visual>
-  <inertial>
-    <origin xyz="0 0 0" rpy="0 ${PI/2} ${PI/2}" />
-    <mass value="${wheelMass}"/>
-    <cylinder_inertia m="${wheelMass}" r="${wheelRadius}" h="${wheelWidth}"/>
-  </inertial>
-</link>
-<gazebo reference="${lr}_wheel">
-  <mu1 value="1.0"/>
-  <mu2 value="1.0"/>
-  <kp  value="10000000.0" />
-  <kd  value="1.0" />
-  <fdir1 value="1 0 0"/>
-  <material>Gazebo/Black</material>
-</gazebo>
-<joint name="${lr}_wheel_hinge" type="continuous">
-  <parent link="chassis"/>
-  <child link="${lr}_wheel"/>
-<origin xyz="${-wheelPos+chassisLength/2} ${tY*wheelWidth/2+tY*chassisWidth/2} ${wheelRadius}" rpy="0 0 0" />
-  <axis xyz="0 1 0" rpy="0 0 0" />
-  <limit effort="100" velocity="100"/>
-  <joint_properties damping="0.0" friction="0.0"/>
-</joint>
-<transmission name="${lr}_trans">
-  <type>transmission_interface/SimpleTransmission</type>
-  <joint name="${lr}_wheel_hinge"/>
-  <actuator name="${lr}Motor">
-    <hardwareInterface>EffortJointInterface</hardwareInterface>
-    <mechanicalReduction>10</mechanicalReduction>
-  </actuator>
-</transmission>
+  <link name="${lr}_wheel">
+    <collision>
+      <origin xyz="0 0 0" rpy="0 ${PI/2} ${PI/2}" />
+      <geometry>
+	<cylinder length="${wheelWidth}" radius="${wheelRadius}"/>
+      </geometry>
+    </collision>
+    <visual>
+      <origin xyz="0 0 0" rpy="0 ${PI/2} ${PI/2}" />
+      <geometry>
+	<cylinder length="${wheelWidth}" radius="${wheelRadius}"/>
+      </geometry>
+      <material name="black"/>
+    </visual>
+    <inertial>
+      <origin xyz="0 0 0" rpy="0 ${PI/2} ${PI/2}" />
+      <mass value="${wheelMass}"/>
+      <cylinder_inertia m="${wheelMass}" r="${wheelRadius}" h="${wheelWidth}"/>
+    </inertial>
+  </link>
+  <gazebo reference="${lr}_wheel">
+    <mu1 value="1.0"/>
+    <mu2 value="1.0"/>
+    <kp  value="10000000.0" />
+    <kd  value="1.0" />
+    <fdir1 value="1 0 0"/>
+    <material>Gazebo/Black</material>
+  </gazebo>
+  <joint name="${lr}_wheel_hinge" type="continuous">
+    <parent link="chassis"/>
+    <child link="${lr}_wheel"/>
+  <origin xyz="${-wheelPos+chassisLength/2} ${tY*wheelWidth/2+tY*chassisWidth/2} ${wheelRadius}" rpy="0 0 0" />
+    <axis xyz="0 1 0" rpy="0 0 0" />
+    <limit effort="100" velocity="100"/>
+    <joint_properties damping="0.0" friction="0.0"/>
+  </joint>
+  <transmission name="${lr}_trans">
+    <type>transmission_interface/SimpleTransmission</type>
+    <joint name="${lr}_wheel_hinge">
+      <hardwareInterface>EffortJointInterface</hardwareInterface>
+    </joint>
+    <actuator name="${lr}Motor">
+      <hardwareInterface>EffortJointInterface</hardwareInterface>
+      <mechanicalReduction>10</mechanicalReduction>
+    </actuator>
+  </transmission>
 </macro>
 </robot>

File: mybot_description/urdf/materials.xacro (robot description, xacro)
@@ -1,2 +1,3 @@
+<?xml version="1.0"?>
 <robot>
 <material name="black">

File: mybot_description/urdf/mybot.xacro (robot description, xacro)
@@ -43,5 +43,44 @@
   </inertial>
 </link>
+<joint name="fixed" type="fixed">
+  <parent link="chassis"/>
+  <child link="caster_wheel"/>
+</joint>
+<link name="caster_wheel">
+  <collision>
+    <origin xyz="${casterRadius-chassisLength/2} 0 ${casterRadius-chassisHeight+wheelRadius}" rpy="0 0 0"/>
+    <geometry>
+      <sphere radius="${casterRadius}"/>
+    </geometry>
+  </collision>
+  <visual>
+    <origin xyz="${casterRadius-chassisLength/2} 0 ${casterRadius-chassisHeight+wheelRadius}" rpy="0 0 0"/>
+    <geometry>
+      <sphere radius="${casterRadius}"/>
+    </geometry>
+    <material name="red"/>
+  </visual>
+  <inertial>
+    <origin xyz="${casterRadius-chassisLength/2} 0 ${casterRadius-chassisHeight+wheelRadius}" rpy="0 0 0"/>
+    <mass value="${casterMass}"/>
+    <sphere_inertia m="${casterMass}" r="${casterRadius}"/>
+  </inertial>
+</link>
 <wheel lr="left" tY="1"/>
 <wheel lr="right" tY="-1"/>
+<include>
+  <uri>model://hokuyo</uri>
+  <pose>0.2 0 0.2 0 0 0</pose>
+</include>
+<joint name="hokuyo_joint" type="revolute">
+  <child>hokuyo::link</child>
+  <parent>chassis</parent>
+  <axis>
+    <xyz>0 0 1</xyz>
+    <limit>
+      <upper>0</upper>
+      <lower>0</lower>
+    </limit>
+  </axis>
+</joint>
 </robot>

Commit message: updated changes

File: mybot_description/urdf/macros.xacro (robot description, xacro)
@@ -19,5 +19,5 @@
   />
 </macro>
-<macro name="wheel" params="lr tY">
+<macro name="wheel" params="lr tX tY">
   <link name="${lr}_wheel">
     <collision>
@@ -41,4 +41,5 @@
   </link>
   <gazebo reference="${lr}_wheel">
+<!--
     <mu1 value="1.0"/>
     <mu2 value="1.0"/>
@@ -46,4 +47,5 @@
     <kd  value="1.0" />
     <fdir1 value="1 0 0"/>
+    -->
     <material>Gazebo/Black</material>
   </gazebo>
@@ -51,5 +53,6 @@
     <parent link="chassis"/>
     <child link="${lr}_wheel"/>
-  <origin xyz="${-wheelPos+chassisLength/2} ${tY*wheelWidth/2+tY*chassisWidth/2} ${wheelRadius}" rpy="0 0 0" />
+    <!--    <origin xyz="${tX*chassisLength/2} ${tY*wheelWidth/2+tY*chassisWidth/2} ${wheelRadius}" rpy="0 0 0" /> -->
+    <origin xyz="${tX*chassisLength/2} ${tY*chassisWidth/2} ${wheelRadius}" rpy="0 0 0" />
     <axis xyz="0 1 0" rpy="0 0 0" />
     <limit effort="100" velocity="100"/>

File: mybot_description/urdf/mybot.xacro (robot description, xacro)
@@ -3,12 +3,11 @@
         <!-- Put here the robot description -->
 <xacro:property name="PI" value="3.1415926535897931"/>
-<xacro:property name="chassisHeight" value="0.1"/>
+<xacro:property name="chassisHeight" value="0.1" />
 <xacro:property name="chassisLength" value="0.4"/>
 <xacro:property name="chassisWidth" value="0.2"/>
 <xacro:property name="chassisMass" value="50"/>
-<xacro:property name="casterRadius" value="0.05"/>
-<xacro:property name="casterMass" value="5"/>
-<xacro:property name="wheelWidth" value="0.05"/>
-<xacro:property name="wheelRadius" value="0.1"/>
+<xacro:property name="laserPosHeight" value="0.15"/>
+<xacro:property name="wheelWidth" value="0.02"/>
+<xacro:property name="wheelRadius" value="0.05"/>
 <xacro:property name="wheelPos" value="0.2"/>
 <xacro:property name="wheelMass" value="5"/>
@@ -18,12 +17,14 @@
 <xacro:include filename="$(find mybot_description)/urdf/materials.xacro" />
 <xacro:include filename="$(find mybot_description)/urdf/macros.xacro" />
-<link name="footprint" />
+<link name="base_link" />
 <joint name="base_joint" type="fixed">
-  <parent link="footprint"/>
+  <parent link="base_link"/>
   <child link="chassis"/>
+  <origin xyz="${-chassisLength/2} 0 0" rpy="0 0 0" />
+  <axis xyz="1 0 0" rpy="0 0 0" />
 </joint>
 <link name='chassis'>
   <collision>
-    <origin xyz="0 0 ${wheelRadius}" rpy="0 0 0"/>
+    <origin xyz="0 0 ${wheelRadius+chassisHeight/2}" rpy="0 0 0"/>
     <geometry>
       <box size="${chassisLength} ${chassisWidth} ${chassisHeight}"/>
@@ -31,5 +32,5 @@
   </collision>
   <visual>
-    <origin xyz="0 0 ${wheelRadius}" rpy="0 0 0"/>
+    <origin xyz="0 0 ${wheelRadius+chassisHeight/2}" rpy="0 0 0"/>
     <geometry>
       <box size="${chassisLength} ${chassisWidth} ${chassisHeight}"/>
@@ -38,49 +39,38 @@
   </visual>
   <inertial>
-    <origin xyz="0 0 ${wheelRadius}" rpy="0 0 0"/>
+    <origin xyz="0 0 ${wheelRadius+chassisHeight/2}" rpy="0 0 0"/>
     <mass value="${chassisMass}"/>
     <box_inertia m="${chassisMass}" x="${chassisLength}" y="${chassisWidth}" z="${chassisHeight}"/>
   </inertial>
 </link>
-<joint name="fixed" type="fixed">
-  <parent link="chassis"/>
-  <child link="caster_wheel"/>
+<wheel lr="left_front" tX="0.6" tY="1"/>
+<wheel lr="right_front" tX="0.6" tY="-1"/>
+<wheel lr="left_back" tX="-0.6" tY="1"/>
+<wheel lr="right_back" tX="-0.6" tY="-1"/>
+<joint name="hokuyo_joint" type="fixed">
+  <axis xyz="0 1 0" />
+  <origin xyz="0 0 ${laserPosHeight}" rpy="0 0 0"/>
+  <parent link="base_link"/>
+  <child link="hokuyo_link"/>
 </joint>
-<link name="caster_wheel">
+<!-- Hokuyo Laser -->
+<link name="hokuyo_link">
   <collision>
-    <origin xyz="${casterRadius-chassisLength/2} 0 ${casterRadius-chassisHeight+wheelRadius}" rpy="0 0 0"/>
+    <origin xyz="0 0 0" rpy="0 0 0"/>
     <geometry>
-      <sphere radius="${casterRadius}"/>
+  <box size="0.1 0.1 0.1"/>
     </geometry>
   </collision>
   <visual>
-    <origin xyz="${casterRadius-chassisLength/2} 0 ${casterRadius-chassisHeight+wheelRadius}" rpy="0 0 0"/>
+    <origin xyz="0 0 0" rpy="0 0 0"/>
     <geometry>
-      <sphere radius="${casterRadius}"/>
+      <mesh filename="/home/tdvu/.gazebo/models/hokuyo/meshes/hokuyo.dae"/>
     </geometry>
-    <material name="red"/>
   </visual>
   <inertial>
-    <origin xyz="${casterRadius-chassisLength/2} 0 ${casterRadius-chassisHeight+wheelRadius}" rpy="0 0 0"/>
-    <mass value="${casterMass}"/>
-    <sphere_inertia m="${casterMass}" r="${casterRadius}"/>
+    <mass value="1e-5" />
+    <origin xyz="0 0 0" rpy="0 0 0"/>
+    <inertia ixx="1e-6" ixy="0" ixz="0" iyy="1e-6" iyz="0" izz="1e-6" />
   </inertial>
 </link>
-<wheel lr="left" tY="1"/>
-<wheel lr="right" tY="-1"/>
-<include>
-  <uri>model://hokuyo</uri>
-  <pose>0.2 0 0.2 0 0 0</pose>
-</include>
-<joint name="hokuyo_joint" type="revolute">
-  <child>hokuyo::link</child>
-  <parent>chassis</parent>
-  <axis>
-    <xyz>0 0 1</xyz>
-    <limit>
-      <upper>0</upper>
-      <lower>0</lower>
-    </limit>
-  </axis>
-</joint>
 </robot>

Commit message: updated changes

File: mybot_description/urdf/macros.xacro (robot description, xacro)
@@ -50,5 +50,5 @@
     <material>Gazebo/Black</material>
   </gazebo>
-  <joint name="${lr}_wheel_hinge" type="continuous">
+  <joint name="${lr}_wheel_joint" type="continuous">
     <parent link="chassis"/>
     <child link="${lr}_wheel"/>
@@ -61,5 +61,5 @@
   <transmission name="${lr}_trans">
     <type>transmission_interface/SimpleTransmission</type>
-    <joint name="${lr}_wheel_hinge">
+    <joint name="${lr}_wheel_joint">
       <hardwareInterface>EffortJointInterface</hardwareInterface>
     </joint>

File: mybot_description/urdf/mybot.xacro (robot description, xacro)
@@ -44,16 +44,16 @@
   </inertial>
 </link>
-<wheel lr="left_front" tX="0.6" tY="1"/>
-<wheel lr="right_front" tX="0.6" tY="-1"/>
-<wheel lr="left_back" tX="-0.6" tY="1"/>
-<wheel lr="right_back" tX="-0.6" tY="-1"/>
-<joint name="hokuyo_joint" type="fixed">
+<wheel lr="front_left" tX="0.6" tY="1"/>
+<wheel lr="front_right" tX="0.6" tY="-1"/>
+<wheel lr="back_left" tX="-0.6" tY="1"/>
+<wheel lr="back_right" tX="-0.6" tY="-1"/>
+<joint name="laser_joint" type="fixed">
   <axis xyz="0 1 0" />
   <origin xyz="0 0 ${laserPosHeight}" rpy="0 0 0"/>
   <parent link="base_link"/>
-  <child link="hokuyo_link"/>
+  <child link="laser"/>
 </joint>
 <!-- Hokuyo Laser -->
-<link name="hokuyo_link">
+<link name="laser">
   <collision>
     <origin xyz="0 0 0" rpy="0 0 0"/>
@@ -65,5 +65,5 @@
     <origin xyz="0 0 0" rpy="0 0 0"/>
     <geometry>
-      <mesh filename="/home/tdvu/.gazebo/models/hokuyo/meshes/hokuyo.dae"/>
+      <mesh filename="package://mybot_description/meshes/hokuyo.dae"/>
     </geometry>
   </visual>
